File: PCB_Sensemat_Final/PCB_Sensemat_Final.kicad_sch (KiCad schematic)
At the start: 53 parts, among them J1 teensy_ingangen_1tm24_Socket, J2 Philips_pins_1tm24, J3 Philips_pins_30tm53, J4 teensy_ingangen_25tm48_Socket, U4 DAC0_MCP4725, U5 DAC1_MCP4725, U6 Teensy4.1, U7 ADS131M08xPBS, Y1 ASE-xxxMHz

Commit message: PCB_Sensemat
Parts:
- C25: LCSC C1785 -> C107107
Changed lines of the file:
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@@
 			)
 		)
-		(property "LCSC" "C1785"
+		(property "LCSC" "C107107"
 			(at 64.4652 165.1 0)
 			(hide yes)
