File: PCB_Sensemat_Final/PCB_Sensemat_Final.kicad_pcb (KiCad board)
At the start: 4 copper layers, 70 x 65 mm, 53 parts, among them J1 teensy_ingangen_1tm24_Socket, J2 Philips_pins_1tm24, J3 Philips_pins_30tm53, J4 teensy_ingangen_25tm48_Socket, U4 DAC0_MCP4725, U5 DAC1_MCP4725, U7 ADS131M08xPBS, Y1 ASE-xxxMHz

Commit message: PCB_Sensemat
Routing:
- net /ADC_MISO: track 83.3 -> 86.7 mm
- net /ADC_MOSI: track 83.2 -> 85.4 mm
- net /ADC_CS: track 75.3 -> 77.1 mm

Commit message: Final production version
Other:
- board size 70 x 65 mm -> 73.4 x 69.5 mm
Changed lines of the file:
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@@
 	)
 	(gr_rect
-		(start 76.4 57.05)
-		(end 146.4 122.05)
+		(start 74.8 55)
+		(end 148.2 124.45)
 		(radius 2)
 		(stroke
@@
 		(polygon
 			(pts
-				(xy 75.95 56.45) (xy 146.8 56.6) (xy 146.9 122.3) (xy 75.95 122.3) (xy 75.85 56.45)
+				(xy 73 54.15) (xy 149.15 54.25) (xy 149.05 125.15) (xy 73.15 125.35) (xy 73 57.1)
 			)
 		)
@@
 		(polygon
 			(pts
-				(xy 76 56.45) (xy 146.95 56.6) (xy 146.95 122.55) (xy 76 122.4) (xy 75.75 56.3)
+				(xy 72.3 53.9) (xy 148.949872 54.104924) (xy 148.747031 125.850058) (xy 71.75521 125.645155) (xy 72.245943 74.835503)
 			)
 		)
